Commit message: updated iiwa urdf + fixes

File: KUKA-iiwa-insertion/kuka_iiwa_insertion/robot/urdf/iiwa14.urdf (robot description, URDF)
Before this commit: robot iiwa14, 10 links, 9 joints
Links:
- link iiwa_link_0: geometry collision mesh filename=../meshes/collision/link_0.stl; visual mesh filename=../meshes/visual/link_0.stl
- link iiwa_link_1: geometry collision mesh filename=../meshes/collision/link_1.stl; visual mesh filename=../meshes/visual/link_1.stl
- link iiwa_link_2: geometry collision mesh filename=../meshes/collision/link_2.stl; visual mesh filename=../meshes/visual/link_2.stl
- link iiwa_link_3: geometry collision mesh filename=../meshes/collision/link_3.stl; visual mesh filename=../meshes/visual/link_3.stl
- link iiwa_link_4: geometry collision mesh filename=../meshes/collision/link_4.stl; visual mesh filename=../meshes/visual/link_4.stl
- link iiwa_link_5: geometry collision mesh filename=../meshes/collision/link_5.stl; visual mesh filename=../meshes/visual/link_5.stl
- link iiwa_link_6: geometry collision mesh filename=../meshes/collision/link_6.stl; visual mesh filename=../meshes/visual/link_6.stl
- link iiwa_link_7: geometry collision mesh filename=../meshes/collision/link_7.stl; visual mesh filename=../meshes/visual/link_7.stl
